File: hw/alarm/alarm.kicad_pcb (KiCad board)
At the start: 2 copper layers, 105 x 73 mm, 54 parts, among them IC1 DS3231S#T&R, IC2 TSOP38238, IC3 SHT40-BD1B-R2, IC4 23K256-I_SN, IC5 PEC11S-929K-S0015, J1 4328, J2 SFV24R-4STBE1HLF, Q1 DMG2305UX-7, Q3 Si1308EDL-T1-GE3, U1 RaspberryPi_Pico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

Commit message: Finish board layout initial ver
Parts:
- removed LS3: PT-1241PFQ, SamacSys_Parts:PT1241PFQ
- added TP1: TestPoint, TestPoint:TestPoint_Pad_1.0x1.0mm, F.Cu at (177.5, 63.0)
- added TP2: TestPoint, TestPoint:TestPoint_Pad_1.0x1.0mm, F.Cu at (180.0, 63.0)
- added TP3: TestPoint, TestPoint:TestPoint_Pad_1.0x1.0mm, F.Cu at (175.0, 63.0)
- added TP4: TestPoint, TestPoint:TestPoint_Pad_1.0x1.0mm, F.Cu at (172.5, 63.0)
- added TP5: TestPoint, TestPoint:TestPoint_Pad_1.0x1.0mm, F.Cu at (170.0, 63.0)
- LS1, LS2: value PT-1241PFQ -> CPT-9019A-SMT-TR; footprint SamacSys_Parts:PT1241PFQ -> CPT_9019A_SMT_TR:CPT-9019A_CUD; moved to F.Cu
- U1: footprint Module_RaspberryPi_Pico:RaspberryPi_Pico_Original_SMD_MountingHoles_HandSolder_Castellated -> Module_RaspberryPi_Pico:RaspberryPi_Pico_Original_SMD
- moved LS1 56.2 mm to (113.5, 123.0), turned to -90 degrees
- moved LS2 53.4 mm to (101.5, 123.0), turned to -90 degrees
- moved J1 48.9 mm to (178.5, 95.3), turned to 0 degrees
- moved C1 39.8 mm to (111.5, 64.5)
- moved IC4 39.8 mm to (105.0, 66.0)
- moved IC3 23.5 mm to (111.9, 105.2), turned to -90 degrees
- moved C2 19.7 mm to (94.5, 106.0), turned to -90 degrees
- moved C15 17.6 mm to (112.0, 109.4), turned to 180 degrees
- moved C11 16.5 mm to (111.5, 71.5)
- moved D4 11.4 mm to (103.5, 74.5), turned to 90 degrees
- moved D3 6.82 mm to (103.5, 80.0), turned to 90 degrees
- moved IC1 6.50 mm to (102.5, 108.5), turned to 0 degrees
- moved C4 5.36 mm to (108.0, 74.8)
- moved R1 5.32 mm to (108.0, 90.0), turned to 180 degrees
- moved C3 5.06 mm to (108.0, 72.5)
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Connections:
- LS1 pad 1: GND -> Net-(U1-GPIO16)
- LS1 pad 2: Net-(LS1-+) -> GND
- LS2 pad 1: GND -> Net-(U1-GPIO17)
- LS2 pad 2: Net-(LS2-+) -> GND
- U1 pad 21: Net-(LS3-+) -> Net-(U1-GPIO16)
- U1 pad 22: Net-(LS2-+) -> Net-(U1-GPIO17)
- U1 pad 24: Net-(LS1-+) -> unconnected-(U1-GPIO18-Pad24)
- U1 pad TP1: (no net) -> Net-(U1-USB_GND)
- U1 pad TP2: (no net) -> Net-(U1-USB_DM)
- U1 pad TP3: (no net) -> Net-(U1-USB_DP)
- U1 pad TP4: (no net) -> unconnected-(U1-~{SMPS_PS}-PadTP4)
- U1 pad TP5: (no net) -> Net-(U1-LED_OUT)
- U1 pad TP6: (no net) -> Net-(U1-~{BOOTSEL})
Routing:
- net GND: track 3.69 -> 147.6 mm, vias 0 -> 18
- net /MOSI: track 0.00 -> 114.1 mm, vias 0 -> 3
- net /SCL: track 6.18 -> 117.3 mm, vias 0 -> 3
- net /SCK: track 0.00 -> 105.1 mm, vias 0 -> 1
- net /MISO: track 0.00 -> 95.5 mm, vias 0 -> 1
- net /SRAMCS: track 0.00 -> 85.9 mm, vias 0 -> 3
- net Net-(Q1-D): track 0.00 -> 85.5 mm
- net /SDA: track 8.66 -> 89.4 mm, vias 0 -> 4
- net +3.3V: track 18.8 -> 97.7 mm, vias 0 -> 4
- net Net-(U1-GPIO17): track 0.00 -> 76.7 mm, vias 0 -> 1
- net /DC: track 0.00 -> 71.0 mm, vias 0 -> 1
- net /EinkCS: track 0.00 -> 61.4 mm, vias 0 -> 1
- net Net-(U1-GPIO16): track 0.00 -> 60.9 mm, vias 0 -> 1
- net Net-(IC2-OUT): track 3.27 -> 60.3 mm, vias 0 -> 1
- net /EinkBUSY: track 0.00 -> 56.6 mm, vias 0 -> 1
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- added copper zone on F.Cu, net +3.3V
