File: hw/front_plate/front_plate.kicad_pcb (KiCad board)
At the start: 2 copper layers, 77 x 79 mm, 27 parts

Commit message: Add front and rear plate
Other:
- board text added: "3.3V"
- board text added: "GP14"
- board text added: "GP6"
- board text added: "GP7"
- board text added: "GP8"
- board text added: "GP9"
- board text added: "i2c"
- board text added: "persuasive_waker v3 Ben Bokser"
Changed lines of the file:
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@@
+	)
+	(gr_line
+		(start 161.25 53)
+		(end 161.25 52)
+		(stroke
+			(width 0.2)
+			(type default)
+		)
+		(layer "F.SilkS")
+	)
+	(gr_line
+		(start 144.25 53)
+		(end 161.25 53)
+		(stroke
+			(width 0.2)
+			(type default)
+		)
+		(layer "F.SilkS")
+	)
+	(gr_line
+		(start 171 53)
+		(end 171 52)
+		(stroke
+			(width 0.2)
+			(type default)
+		)
+		(layer "F.SilkS")
+	)
+	(gr_line
+		(start 162 53)
+		(end 162 52)
+		(stroke
+			(width 0.2)
+			(type default)
+		)
+		(layer "F.SilkS")
+	)
+	(gr_line
+		(start 162 53)
+		(end 171 53)
+		(stroke
+			(width 0.2)
+			(type default)
+		)
+		(layer "F.SilkS")
+	)
+	(gr_line
+		(start 144.25 53)
+		(end 144.25 52)
+		(stroke
+			(width 0.2)
+			(type default)
+		)
+		(layer "F.SilkS")
 	)
 	(gr_line
@@
 		(layer "Edge.Cuts")
 	)
+	(gr_text "GP7"
+		(at 157.25 56.25 90)
+		(layer "F.SilkS")
+		(effects
+			(font
+				(size 1 1)
+				(thickness 0.25)
+				(bold yes)
+			)
+			(justify left bottom)
+		)
+	)
+	(gr_text "GP9"
+		(at 152.25 56.25 90)
+		(layer "F.SilkS")
+		(effects
+			(font
+				(size 1 1)
+				(thickness 0.25)
+				(bold yes)
+			)
+			(justify left bottom)
+		)
+	)
+	(gr_text "3.3V"
+		(at 147.25 56.75 90)
+		(layer "F.SilkS")
+		(effects
+			(font
+				(size 1 1)
+				(thickness 0.25)
+				(bold yes)
+			)
+			(justify left bottom)
+		)
+	)
+	(gr_text "GP8"
+		(at 154.75 56.25 90)
+		(layer "F.SilkS")
+		(effects
+			(font
+				(size 1 1)
+				(thickness 0.25)
+				(bold yes)
+			)
+			(justify left bottom)
+		)
+	)
+	(gr_text "i2c"
+		(at 165.25 55 0)
+		(layer "F.SilkS")
+		(effects
+			(font
+				(size 1 1)
+				(thickness 0.25)
+				(bold yes)
+			)
+			(justify left bottom)
+		)
+	)
+	(gr_text "GP6"
+		(at 159.75 56.25 90)
+		(layer "F.SilkS")
+		(effects
+			(font
+				(size 1 1)
+				(thickness 0.25)
+				(bold yes)
+			)
+			(justify left bottom)
+		)
+	)
+	(gr_text "persuasive_waker v3\nBen Bokser"
+		(at 116 127.25 0)
+		(layer "F.SilkS")
+		(effects
+			(font
+				(size 1.5 1.5)
+				(thickness 0.3)
+				(bold yes)
+			)
+			(justify left bottom)
+		)
+	)
+	(gr_text "GP14"
+		(at 149.75 57.25 90)
+		(layer "F.SilkS")
+		(effects
+			(font
+				(size 1 1)
+				(thickness 0.25)
+				(bold yes)
+			)
+			(justify left bottom)
+		)
+	)
 )
